File: pcb/pcb/pcb.kicad_sch (KiCad schematic)
At the start: 72 parts, among them J1 Conn_01x03_Pin, J10 Conn_01x03_Pin, J11 Conn_01x03_Pin, J12 Conn_01x03_Pin, J13 Conn_01x03_Pin, J14 Conn_01x03_Pin, J15 Conn_01x03_Pin, J16 Conn_01x03_Pin, J17 Conn_01x03_Pin, J18 Conn_01x04_Pin, J2 Conn_01x03_Pin, J20 Conn_01x08_Socket, J3 Conn_01x03_Pin, J4 Conn_01x03_Pin, J5 Conn_01x03_Pin, J6 Conn_01x03_Pin, J7 Conn_01x03_Pin, J8 Conn_01x03_Pin, J9 Conn_01x03_Pin, U1 Pico, U2 4052, U3 4052, U4 LM324

Commit message: Final PCB revision, i guess?
Parts:
- added C15, C16, C17, C18, C19, C20, C21, C22, C23, C24: C, Capacitor_SMD:C_0805_2012Metric, symbol Device:C
- added NT3: NetTie_2, NetTie:NetTie-2_SMD_Pad0.5mm, symbol Device:NetTie_2
- JP1: now left out of the parts list
Connections:
- net +5V: now also C20.1, C21.1, C22.1, C23.1, C24.1
- net +5VP: now also C15.1, C16.1, C17.1, C18.1, C19.1
- net GND: now also C20.2, C21.2, C22.2, C23.2, C24.2, NT3.1
- net GNDPWR: now also C15.2, C16.2, C17.2, C18.2, C19.2, NT3.2
Other:
- moved on the sheet: C1, C14, NT1, NT2
